Commit message: Enhance URDF with collision and inertial data
Added collision and inertial properties for each link in the robot model.

File: Mes_codes/robot5DoF.urdf (robot description, URDF)
Before this commit: robot dh_5dof_robot, 6 links, 5 joints
Links:
- link base_link: mass None -> 2.0; geometry collision cylinder length=0.05 radius=0.10; visual cylinder length=0.05 radius=0.10
- link link_1: mass None -> 0.40; geometry collision cylinder length=0.10 radius=0.04; visual cylinder length=0.10 radius=0.04
- link link_2: mass None -> 0.60; geometry collision box size=0.06 0.06 0.20; visual cylinder length=0.20 radius=0.03
- link link_3: mass None -> 0.35; geometry collision box size=0.05 0.05 0.10; visual cylinder length=0.10 radius=0.025
- link link_4: mass None -> 0.20; geometry collision cylinder length=0.05 radius=0.02; visual cylinder length=0.05 radius=0.02
- link link_5: mass None -> 0.10; geometry collision box size=0.02 0.02 0.01; visual box size=0.02 0.02 0.01
Joints:
- joint joint_1: limit lower=-3.14 upper=3.14 effort=100 velocity=1.0 -> lower=-3.1416 upper=3.1416 effort=0.45 velocity=6
- joint joint_2: axis 0 0 1 -> 0 1 0; limit lower=-3.14 upper=3.14 effort=100 velocity=1.0 -> lower=-3.1416 upper=3.1416 effort=0.45 velocity=6; origin xyz=0 0 0 rpy=1.57079632679 0 0 -> xyz=0 0 0.05 rpy=0 0 0
- joint joint_3: axis 0 0 1 -> 0 1 0; limit lower=-3.14 upper=3.14 effort=100 velocity=1.0 -> lower=-3.1416 upper=3.1416 effort=0.45 velocity=6; origin xyz=0.2 0 0 rpy=0 0 0 -> xyz=0 0 0.20 rpy=0 0 0
- joint joint_4: axis 0 0 1 -> 0 1 0; limit lower=-3.14 upper=3.14 effort=100 velocity=1.0 -> lower=-3.1416 upper=3.1416 effort=0.45 velocity=6; origin xyz=0.1 0 0.01 rpy=0 0 0 -> xyz=0 0 0.10 rpy=0 0 0
- joint joint_5: limit lower=-3.14 upper=3.14 effort=100 velocity=1.0 -> lower=-3.1416 upper=3.1416 effort=0.45 velocity=6; origin xyz=0 0 0 rpy=1.57079632679 0 0 -> xyz=0 0 0.05 rpy=0 0 0
